File: PCB/PCB.kicad_pcb (KiCad board)
At the start: 2 copper layers, 39 x 46 mm, 10 parts, among them J1 Conn_01x02, J2 Conn_01x02, SW1 SW_MEC_5E, SW2 SW_MEC_5E, SW3 SW_MEC_5E, SW4 SW_DPDT_x2, U1 ESP32-c3, U2 MPU6050_PCB

Commit message: feat: driver proj created
Other:
- board text added: "Snímač gest M1I2"
- board text removed: "Snímač gest M1I1"

Commit message: feat: zaverecna zprava, pcb m2 WIP
Parts:
- removed D2: LED, LED_THT:LED_Oval_W5.2mm_H3.8mm
- removed SW3: SW_MEC_5E, Tlacitka:Arduino_tlacitko
- removed SW4: SW_DPDT_x2, Tlacitka:KLS_on_on_moje
- added R1: 100k, Resistor_THT:R_Axial_DIN0207_L6.3mm_D2.5mm_P7.62mm_Horizontal, F.Cu at (-468.2, -203.0)
- added R2: 100k, Resistor_THT:R_Axial_DIN0207_L6.3mm_D2.5mm_P7.62mm_Horizontal, F.Cu at (-468.2, -198.9)
- added U3: ~, nabijecky_moje_pcb:TP4056, F.Cu at (-453.8, -193.8)
- SW2: value SW_MEC_5E -> SW_DPDT_x2; footprint Tlacitka:Arduino_tlacitko -> Tlacitka:KLS_on_on_moje
- moved U1 359.1 mm to (-460.3, -227.0)
- moved U2 354.3 mm to (-456.1, -230.2), turned to 0 degrees
- moved SW1 349.0 mm to (-476.1, -203.2), turned to 0 degrees
- moved SW2 343.2 mm to (-436.6, -229.0), turned to 0 degrees
- moved J2 342.6 mm to (-424.8, -217.8), turned to 0 degrees
- moved D1 341.6 mm to (-467.6, -194.2)
- moved J1 309.3 mm to (-438.2, -218.0), turned to 0 degrees
Connections:
- J2 pad 1: GND -> Net-(J2-Pin_1)
- SW2 pad 1: Net-(SW2-Pad1) -> VCC
- SW2 pad 2: unconnected-(SW2-Pad2) -> Net-(SW2A-B)
- U1 pad 10: Net-(SW1-Pad1) -> unconnected-(U1-Pad10)
- U1 pad 20: Net-(SW2-Pad1) -> unconnected-(U1-Pad20)
- U1 pad 21: Net-(SW3-Pad1) -> Net-(SW1-Pad1)
- U1 pad 5: unconnected-(U1-Pad5) -> Net-(R1-Pad2)
- U1 pad 6: unconnected-(U1-Pad6) -> Net-(R1-Pad1)
Routing:
- net Net-(J1-Pin_2): track 88.8 -> 0.00 mm
- net VCC: track 82.0 -> 0.00 mm
- net Net-(D1-A): track 65.9 -> 0.00 mm
- net Net-(SW2-Pad1): track 23.9 -> 0.00 mm
- net Net-(SW1-Pad1): track 18.6 -> 0.00 mm
- net Net-(SW3-Pad1): track 12.6 -> 0.00 mm
- net Net-(J2-Pin_2): track 8.86 -> 0.00 mm
- net Net-(U2-INT): track 7.15 -> 0.00 mm
- net Net-(U1-SDA): track 5.32 -> 0.00 mm
- net Net-(U1-SCL): track 5.32 -> 0.00 mm
Other:
- board outline removed
- board text removed: "Snímač gest M1I2"

Commit message: feat: pcb model 2 gerbers
Parts:
- moved U1 95.9 mm to (-364.9, -237.0)
- moved D1 95.8 mm to (-373.7, -213.0)
- moved R2 91.4 mm to (-377.5, -210.5), turned to 180 degrees
- moved R1 83.8 mm to (-385.1, -214.0)
- moved SW1 83.4 mm to (-393.0, -210.5), turned to 180 degrees
- moved U2 73.3 mm to (-383.5, -219.8), turned to 180 degrees
- moved SW2 72.3 mm to (-366.1, -212.8)
- moved J2 59.9 mm to (-367.2, -201.0), turned to 90 degrees
- moved U3 57.9 mm to (-396.0, -191.5)
- moved J1 49.1 mm to (-394.8, -240.8), turned to -90 degrees
Routing:
- net VCC: track 0.00 -> 68.5 mm
- net Net-(J1-Pin_2): track 0.00 -> 68.1 mm
- net Net-(R1-Pad2): track 0.00 -> 28.5 mm
- net Net-(R1-Pad1): track 0.00 -> 25.4 mm
- net Net-(SW1-Pad1): track 0.00 -> 16.5 mm
- net Net-(D1-A): track 0.00 -> 11.4 mm
- net Net-(J2-Pin_1): track 0.00 -> 11.2 mm
- net Net-(SW2A-B): track 0.00 -> 8.63 mm
- net Net-(U2-INT): track 0.00 -> 6.98 mm
- net Net-(J2-Pin_2): track 0.00 -> 6.56 mm
- net Net-(U1-SDA): track 0.00 -> 4.22 mm
- net Net-(U1-SCL): track 0.00 -> 4.22 mm
Other:
- board outline added: 37.5 x 53.5 mm
- board text added: "Snímač gest M2I1"
